File: Kicad/CardSizeMidiController/CardSizeMidiController.kicad_pcb (KiCad board)
At the start: 2 copper layers, 85.7 x 54 mm, 61 parts, among them J1 USB_B, J2 Conn_02x03_Odd_Even, J3 MIDI OUT, J4 AudioJack3, J5 Screw_Terminal_01x01, J6 Screw_Terminal_01x01, J7 Screw_Terminal_01x01, J8 Screw_Terminal_01x01, SW0 SW_Push, SW1 SW_Push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

Commit message: changed caps to smd
Parts:
- C1: value 2.2u -> 100n; footprint Capacitor_THT:CP_Radial_D5.0mm_P2.50mm -> Capacitor_SMD:C_0805_2012Metric_Pad1.15x1.40mm_HandSolder
- C2: value 100u -> 10u; footprint Capacitor_THT:CP_Radial_D6.3mm_P2.50mm -> Capacitor_SMD:C_0805_2012Metric_Pad1.15x1.40mm_HandSolder
- moved C2 6.99 mm to (30.0, 8.00), turned to 45 degrees
- moved C1 6.45 mm to (37.0, 12.0)
Routing:
- net +5V: track 188.1 -> 179.3 mm
- net GND: track 87.7 -> 94.5 mm, vias 1 -> 2
Other:
- board text added: "27"
- board text added: "28"
- board text added: "29"
- board text added: "30"
- board text added: "31"
- board text added: "7 10 1"
- board text added: "CC1 26 CC2 102 103 104 105 112 113 CC3 114 115 116 117 118 119"
- board text added: "LEVEL PAN MOD"
- board text added: "MIDI CC CODES"
- board text removed: "AUTHORIZED SIGNATURE"

Commit message: v0.4
Parts:
- added TP1: TestPoint, TestPoint:TestPoint_Pad_D1.5mm, B.Cu at (2.38, 25.1)
- added TP2: TestPoint, TestPoint:TestPoint_Pad_D1.5mm, B.Cu at (2.38, 20.0)
- added TP3: TestPoint, TestPoint:TestPoint_Pad_D1.5mm, B.Cu at (2.38, 17.5)
- added TP4: TestPoint, TestPoint:TestPoint_Pad_D1.5mm, B.Cu at (2.38, 27.6)
- added TP5: TestPoint, TestPoint:TestPoint_Pad_D1.5mm, B.Cu at (2.38, 22.5)
- added TP6: TestPoint, TestPoint:TestPoint_Pad_D1.5mm, B.Cu at (2.38, 30.2)
- SW0, SW1, SW2, SW3, SW4, SW5: footprint Button_Switch_THT:SW_PUSH_6mm_H5mm -> Button_Switch_SMD:SW_Push_1P1T_NO_6x6mm_H9.5mm
- moved LOGO2 8.70 mm to (4.50, 17.0)
- moved SW1 4.00 mm to (25.0, 47.0)
- moved SW2 4.00 mm to (36.9, 47.0)
- moved SW3 4.00 mm to (48.8, 47.0)
- moved SW4 4.00 mm to (60.7, 47.0)
- moved SW5 4.00 mm to (72.5, 47.0)
- moved SW0 4.00 mm to (13.1, 47.0)
- moved J2 1.60 mm to (3.43, 9.45)
- moved LOGO14 1.60 mm to (1.30, 9.50)
Routing:
- net LED4: track 57.8 -> 92.5 mm, vias 2 -> 0
- net GND: track 94.5 -> 62.4 mm
- net LED1: track 51.0 -> 23.1 mm, vias 0 -> 2
- net +5V: track 179.3 -> 201.3 mm
- net LED5: track 106.1 -> 119.4 mm, vias 1 -> 0
- net MISO: track 95.5 -> 107.4 mm
- net A5: track 79.1 -> 68.9 mm
- net SW0: track 43.1 -> 47.8 mm, vias 1 -> 2
- net ~RST: track 27.5 -> 31.5 mm
- net XTAL1: track 10.6 -> 14.6 mm, vias 0 -> 2
- net LED2: track 30.0 -> 33.6 mm
- net LED0: track 26.4 -> 28.8 mm
- net SW2: track 57.5 -> 59.8 mm, vias 1 -> 2
- net TX: track 42.6 -> 41.0 mm
- net SW1: track 45.3 -> 46.8 mm, vias 1 -> 2
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Other:
- board text added: "GND"
- board text added: "MISO"
- board text added: "MOSI"
- board text added: "RST"
- board text added: "SCK"
- board text added: "Serial number"
- board text added: "VCC"
- board text added: "Version 0.4"
- board text removed: "JLC Order Number"
- board text removed: "Version 0.3"
